File: buffer_overflow.kicad_sch (KiCad schematic)
At the start: 28 parts, among them J1 Barrel_Jack_Switch, J3 NRJ4HF, J4 NRJ4HF, SW1 3PDT, U1 LM741

Commit message: Add Power/LED netclasses and update board
Net classes (Board Setup):
- Power (32 mil): /9V0, /AGND, /PGND, /BAT_GND
- LED (24 mil): /LED*
- Default (14 mil): all other signal nets

Includes accompanying schematic and PCB edits.

Co-Authored-By: Claude Opus 4.8 (1M context) <noreply@anthropic.com>
Parts:
- removed D5: 1N4001, Diode_THT:D_DO-41_SOD81_P10.16mm_Horizontal, symbol Diode:1N4001
- removed J4: NRJ4HF, Connector_Audio:Jack_6.35mm_Neutrik_NRJ4HF_Horizontal, symbol Connector_Audio:NRJ4HF
- removed SW1: 3PDT, symbol Connector_Generic:Conn_01x09
- removed U1: LM741, Package_DIP:DIP-8_W7.62mm_Socket, symbol Amplifier_Operational:LM741
- added C1: 100uF, Capacitor_THT:C_Radial_D8.0mm_H11.5mm_P3.50mm, symbol Device:C_US
- added C2: 100nF, Capacitor_THT:C_Rect_L10.0mm_W2.5mm_P7.50mm_MKS4, symbol Device:C
- added D1: 1N4001, Diode_THT:D_DO-41_SOD81_P10.16mm_Horizontal, symbol Diode:1N4001
- added H1: MountingHole, MountingHole:MountingHole_5.3mm_M5, symbol Mechanical:MountingHole
- added J2: NRJ4HF-1, Connector_Audio:Jack_6.35mm_Neutrik_NRJ4HF_Horizontal, symbol Connector_Audio:NRJ4HF
- added SW1: SW_FSW800_3PDT, edaFactory:SW_FSW800_3PDT, symbol edaFactory:SW_FSW800_3PDT
- added U1: TL071, Package_DIP:DIP-8_W7.62mm, symbol Amplifier_Operational:TL071
- C3: renamed from C2; value C_US -> 10uF
- renumbered C1 to C4, C3 to C5, C4 to C6, C5 to C7, D1 to D2, D2 to D3, D3 to D4, D4 to D5, H1 to H2, H2 to H3
Connections:
- net 9V0: now also D4.2 (A), D5.2 (A), D1.2 (A), U1.7 (V+)
- net AGND: now also J3.S, J2.S, J2.TN; no longer J3.T
- net PGND: now also C1.2, C2.2, SW1.8, U1.4 (V-)
- net LEDK: now reaches D5.1 (K)
- net LEDK: now also D4.1 (K), R9.1
- net BAT_GND: now reaches H3.1, J1.3
- net NINV: now reaches R4.2, R6.1
- net NINV: now also U1.3 (+)
- net at R2.2: now also C1.1, C2.1, D1.1 (K)
- net LEDA: now reaches R9.2
- net LEDA: now also SW1.7; no longer D4.2 (A)
- net 741_Inv renamed INV
- net INV: now also U1.2 (-)
- net 741_OUT renamed OPAMPOUT
- net OPAMPOUT: now also U1.6
- net EFFECT_IN renamed CIRCIN
- net CIRCIN: now also SW1.4
- net EFFECT_OUT renamed CIRCOUT
- net CIRCOUT: now also SW1.1; no longer J3.S
- new net: SW1.3, SW1.6
- new net INPUT_TIP: J2.T, SW1.5
- new net OUT_TIP: J3.T, SW1.2
- no-connect marks 2 -> 3
Other:
- note added: "(misnomer, it's not LEDA)"
- moved on the sheet: D4, D5, H2, H3, J1, J3, R9
