File: buffer_overflow.kicad_pcb (KiCad board)
At the start: 2 copper layers, 52 x 100 mm, 32 parts, among them J1 Barrel_Jack_Switch, J2 NRJ4HF-1, J3 NRJ4HF, SW1 SW_FSW800_3PDT, U1 TL071

Commit message: version sent to JLCPCB 6/4/26
Parts:
- moved C6 1.56 mm to (139.0, 131.0), turned to 90 degrees
Routing:
- net /9V0: track 84.8 -> 71.8 mm
- net /LEDA: track 54.0 -> 64.5 mm
- net Net-(C6-Pad2): track 7.66 -> 4.81 mm
- net /PGND: track 101.3 -> 99.0 mm
- net /OPAMPOUT: track 19.3 -> 20.4 mm
- net /OUT_TIP: track 77.4 -> 78.1 mm
Other:
- board text added: "davidshuman@gmail.com hardware | firmware analog | digital | audio tube amplifiers"
- board text removed: "davidshuman@gmail.com hardware - firmware analog - digital - audio tube amplifiers"
