File: dod250new.kicad_sch (KiCad schematic)
At the start: 31 parts, among them J1 Barrel_Jack_Switch, J2 NRJ4HF-1, J3 NRJ4HF, SW1 SW_FSW800_3PDT, U1 TL071

Commit message: v1.1 sent to JLCPC 6/4/26 evening -- resolved 9V0 battery net disconnect
Parts:
- C1: footprint Capacitor_THT:C_Radial_D8.0mm_H11.5mm_P3.50mm -> Capacitor_THT:CP_Radial_D6.3mm_P2.50mm; Field5 (none) -> ESK107M025AC3AA
- C2: footprint Capacitor_THT:C_Rect_L10.0mm_W2.5mm_P7.50mm_MKS4 -> Capacitor_THT:C_Rect_L7.2mm_W4.5mm_P5.00mm; Field5 (none) -> PHE450KB6100JR05L2
- C4: footprint Capacitor_THT:C_Rect_L10.0mm_W2.5mm_P7.50mm_MKS4 -> Capacitor_THT:C_Rect_L7.2mm_W4.5mm_P5.00mm; Field5 (none) -> PHE450KB4100JR05L2
- C5: footprint Capacitor_THT:C_Rect_L10.0mm_W2.5mm_P7.50mm_MKS4 -> Capacitor_THT:C_Disc_D3.8mm_W2.6mm_P2.50mm; Field5 (none) -> KEMET C315C121J2G5TA
- C6: footprint Capacitor_THT:C_Radial_D5.0mm_H7.0mm_P2.00mm -> Capacitor_THT:CP_Radial_D5.0mm_P2.50mm
- C7: footprint Capacitor_THT:C_Rect_L10.0mm_W2.5mm_P7.50mm_MKS4 -> Capacitor_THT:C_Rect_L7.2mm_W4.5mm_P5.00mm; Field5 (none) -> PHE450KB4010JR05L2
- H2: value MountingHole_Pad -> BATT+
- H3: value MountingHole_Pad -> BATT-
Connections:
- net 9V0: now also C1.1, C2.1, D1.1 (K), R2.2; no longer D1.2 (A), H2.1, J1.1
- new net 9V0_RAW: D1.2 (A), H2.1, J1.1
Changed lines of the file:
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@@
+		)
+	)
+	(label "9V0"
+		(at 76.2 115.57 0)
+		(effects
+			(font
+				(size 1.27 1.27)
+			)
+			(justify left bottom)
 		)
 	)
@@
 		)
 	)
-	(label "9V0"
-		(at 49.53 115.57 0)
-		(effects
-			(font
-				(size 1.27 1.27)
-			)
-			(justify left bottom)
-		)
-	)
 	(label "BAT_GND"
 		(at 49.53 132.08 0)
@@
 		)
 	)
+	(label "9V0_RAW"
+		(at 40.64 115.57 0)
+		(effects
+			(font
+				(size 1.27 1.27)
+			)
+			(justify left bottom)
+		)
+	)
 	(label "PGND"
 		(at 163.83 138.43 0)
@@
 		)
 		(instances
-			(project "buffer_overflow"
+			(project "dod250new"
 				(path "/65eca179-3106-4a88-bde8-4fcb23cd7118"
 					(reference "D5")
@@
 		)
 		(instances
-			(project "buffer_overflow"
+			(project "dod250new"
 				(path "/65eca179-3106-4a88-bde8-4fcb23cd7118"
 					(reference "U1")
@@
 		(in_pos_files yes)
 		(dnp no)
-		(fields_autoplaced yes)
 		(property "Reference" "H3"
 			(at 64.77 130.8099 90)
+			(hide yes)
 			(show_name no)
 			(do_not_autoplace no)
@@
 			)
 		)
-		(property "Value" "MountingHole_Pad"
-			(at 64.77 133.3499 90)
-			(hide yes)
+		(property "Value" "BATT-"
+			(at 63.5 129.54 90)
 			(show_name no)
 			(do_not_autoplace no)
@@
 		)
 		(instances
-			(project "buffer_overflow"
+			(project "dod250new"
 				(path "/65eca179-3106-4a88-bde8-4fcb23cd7118"
 					(reference "H3")
@@
 		)
 		(instances
-			(project "buffer_overflow"
+			(project "dod250new"
 				(path "/65eca179-3106-4a88-bde8-4fcb23cd7118"
 					(reference "RV2")
@@
 		)
 		(instances
-			(project "buffer_overflow"
+			(project "dod250new"
 				(path "/65eca179-3106-4a88-bde8-4fcb23cd7118"
 					(reference "J2")
@@
 		)
 		(instances
-			(project "buffer_overflow"
+			(project "dod250new"
 				(path "/65eca179-3106-4a88-bde8-4fcb23cd7118"
 					(reference "R3")
@@
 			)
 		)
-		(property "Footprint" "Capacitor_THT:C_Radial_D5.0mm_H7.0mm_P2.00mm"
+		(property "Footprint" "Capacitor_THT:CP_Radial_D5.0mm_P2.50mm"
 			(at 175.26 45.72 0)
 			(hide yes)
@@
 		)
 		(instances
-			(project "buffer_overflow"
+			(project "dod250new"
 				(path "/65eca179-3106-4a88-bde8-4fcb23cd7118"
 					(reference "C6")
@@
 			)
 		)
-		(property "Footprint" "Capacitor_THT:C_Rect_L10.0mm_W2.5mm_P7.50mm_MKS4"
+		(property "Footprint" "Capacitor_THT:C_Rect_L7.2mm_W4.5mm_P5.00mm"
 			(at 113.03 44.1452 0)
 			(hide yes)
@@
 			)
 		)
+		(property "Field5" "PHE450KB4100JR05L2"
+			(at 116.84 43.18 90)
+			(hide yes)
+			(show_name no)
+			(do_not_autoplace no)
+			(effects
+				(font
+					(size 1.27 1.27)
+				)
+			)
+		)
 		(pin "1"
 		)
@@
 		)
 		(instances
-			(project "buffer_overflow"
+			(project "dod250new"
 				(path "/65eca179-3106-4a88-bde8-4fcb23cd7118"
 					(reference "C4")
@@
 			)
 		)
-		(property "Footprint" "Capacitor_THT:C_Radial_D8.0mm_H11.5mm_P3.50mm"
+		(property "Footprint" "Capacitor_THT:CP_Radial_D6.3mm_P2.50mm"
 			(at 76.2 125.73 0)
 			(hide yes)
@@
 			)
 		)
+		(property "Field5" "ESK107M025AC3AA"
+			(at 76.2 125.73 0)
+			(hide yes)
+			(show_name no)
+			(do_not_autoplace no)
+			(effects
+				(font
+					(size 1.27 1.27)
+				)
+			)
+		)
 		(pin "1"
 		)
@@
 		)
 		(instances
-			(project "buffer_overflow"
+			(project "dod250new"
 				(path "/65eca179-3106-4a88-bde8-4fcb23cd7118"
 					(reference "C1")
@@
 		)
 		(instances
-			(project "buffer_overflow"
+			(project "dod250new"
 				(path "/65eca179-3106-4a88-bde8-4fcb23cd7118"
 					(reference "R5")
@@
 		)
 		(instances
-			(project "buffer_overflow"
+			(project "dod250new"
 				(path "/65eca179-3106-4a88-bde8-4fcb23cd7118"
 					(reference "D3")
@@
 		)
 		(instances
-			(project "buffer_overflow"
+			(project "dod250new"
 				(path "/65eca179-3106-4a88-bde8-4fcb23cd7118"
 					(reference "RV1")
@@
 		(in_pos_files yes)
 		(dnp no)
-		(fields_autoplaced yes)
 		(property "Reference" "H2"
 			(at 60.96 124.4599 0)
+			(hide yes)
 			(show_name no)
 			(do_not_autoplace no)
@@
 			)
 		)
-		(property "Value" "MountingHole_Pad"
-			(at 60.96 126.9999 0)
-			(hide yes)
+		(property "Value" "BATT+"
+			(at 59.69 123.19 0)
 			(show_name no)
 			(do_not_autoplace no)
@@
 		)
 		(instances
-			(project "buffer_overflow"
+			(project "dod250new"
 				(path "/65eca179-3106-4a88-bde8-4fcb23cd7118"
 					(reference "H2")
@@
 		)
 		(instances
-			(project "buffer_overflow"
+			(project "dod250new"
 				(path "/65eca179-3106-4a88-bde8-4fcb23cd7118"
 					(reference "R8")
@@
 		)
 		(instances
-			(project "buffer_overflow"
+			(project "dod250new"
 				(path "/65eca179-3106-4a88-bde8-4fcb23cd7118"
 					(reference "R6")
@@
 		)
 		(instances
-			(project "buffer_overflow"
+			(project "dod250new"
 				(path "/65eca179-3106-4a88-bde8-4fcb23cd7118"
 					(reference "C3")
@@
 		)
 		(instances
-			(project "buffer_overflow"
+			(project "dod250new"
 				(path "/65eca179-3106-4a88-bde8-4fcb23cd7118"
 					(reference "R9")
@@
 		)
 		(instances
-			(project "buffer_overflow"
+			(project "dod250new"
 				(path "/65eca179-3106-4a88-bde8-4fcb23cd7118"
 					(reference "J3")
@@
 		)
 		(instances
-			(project "buffer_overflow"
+			(project "dod250new"
 				(path "/65eca179-3106-4a88-bde8-4fcb23cd7118"
 					(reference "D2")
@@
 		)
 		(instances
-			(project "buffer_overflow"
+			(project "dod250new"
 				(path "/65eca179-3106-4a88-bde8-4fcb23cd7118"
 					(reference "R7")
@@
 			)
 		)
-		(property "Footprint" "Capacitor_THT:C_Rect_L10.0mm_W2.5mm_P7.50mm_MKS4"
+		(property "Footprint" "Capacitor_THT:C_Disc_D3.8mm_W2.6mm_P2.50mm"
 			(at 151.13 72.0852 0)
 			(hide yes)
@@
 			)
 		)
+		(property "Field5" "KEMET C315C121J2G5TA"
+			(at 154.94 71.12 90)
+			(hide yes)
+			(show_name no)
+			(do_not_autoplace no)
+			(effects
+				(font
+					(size 1.27 1.27)
+				)
+			)
+		)
 		(pin "1"
 		)
@@
 		)
 		(instances
-			(project "buffer_overflow"
+			(project "dod250new"
 				(path "/65eca179-3106-4a88-bde8-4fcb23cd7118"
 					(reference "C5")
@@
 		)
 		(instances
-			(project "buffer_overflow"
+			(project "dod250new"
 				(path "/65eca179-3106-4a88-bde8-4fcb23cd7118"
 					(reference "D1")
@@
 		)
 		(instances
-			(project "buffer_overflow"
+			(project "dod250new"
 				(path "/65eca179-3106-4a88-bde8-4fcb23cd7118"
 					(reference "R1")
@@
 			)
 		)
-		(property "Footprint" "Capacitor_THT:C_Rect_L10.0mm_W2.5mm_P7.50mm_MKS4"
+		(property "Footprint" "Capacitor_THT:C_Rect_L7.2mm_W4.5mm_P5.00mm"
 			(at 216.8652 57.15 0)
 			(hide yes)
@@
 			)
 		)
+		(property "Field5" "PHE450KB4010JR05L2 "
+			(at 215.9 53.34 0)
+			(hide yes)
+			(show_name no)
+			(do_not_autoplace no)
+			(effects
+				(font
+					(size 1.27 1.27)
+				)
+			)
+		)
 		(pin "1"
 		)
@@
 		)
 		(instances
-			(project "buffer_overflow"
+			(project "dod250new"
 				(path "/65eca179-3106-4a88-bde8-4fcb23cd7118"
 					(reference "C7")
@@
 		)
 		(instances
-			(project "buffer_overflow"
+			(project "dod250new"
 				(path "/65eca179-3106-4a88-bde8-4fcb23cd7118"
 					(reference "H1")
@@
 		)
 		(instances
-			(project "buffer_overflow"
+			(project "dod250new"
 				(path "/65eca179-3106-4a88-bde8-4fcb23cd7118"
 					(reference "SW1")
@@
 			)
 		)
-		(property "Footprint" "Capacitor_THT:C_Rect_L10.0mm_W2.5mm_P7.50mm_MKS4"
+		(property "Footprint" "Capacitor_THT:C_Rect_L7.2mm_W4.5mm_P5.00mm"
 			(at 89.2048 129.54 0)
 			(hide yes)
@@
 			)
 		)
+		(property "Field5" "PHE450KB6100JR05L2"
+			(at 90.17 125.73 0)
+			(hide yes)
+			(show_name no)
+			(do_not_autoplace no)
+			(effects
+				(font
+					(size 1.27 1.27)
+				)
+			)
+		)
 		(pin "1"
 		)
@@
 		)
 		(instances
-			(project "buffer_overflow"
+			(project "dod250new"
 				(path "/65eca179-3106-4a88-bde8-4fcb23cd7118"
 					(reference "C2")
@@
 		)
 		(instances
-			(project "buffer_overflow"
+			(project "dod250new"
 				(path "/65eca179-3106-4a88-bde8-4fcb23cd7118"
 					(reference "J1")
@@
 		)
 		(instances
-			(project "buffer_overflow"
+			(project "dod250new"
 				(path "/65eca179-3106-4a88-bde8-4fcb23cd7118"
 					(reference "R4")
@@
 		)
 		(instances
-			(project "buffer_overflow"
+			(project "dod250new"
 				(path "/65eca179-3106-4a88-bde8-4fcb23cd7118"
 					(reference "D4")
@@
 		)
 		(instances
-			(project "buffer_overflow"
+			(project "dod250new"
 				(path "/65eca179-3106-4a88-bde8-4fcb23cd7118"
 					(reference "R2")

Commit message: minor tweaks
Parts:
- H1: value MountingHole -> BatteryLeads
Other:
- company: github.com/whbeers/buffer_overflow -> dod250.shupac.com/v1_1
- title: Buffer Overflow Drive Effect -> DOD Overdrive Preamp 250
- moved on the sheet: C1, C2, C3, C4, C5, C6, C7, D1, D2, D3, D4, D5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
